File: adbee.kicad_pcb (KiCad board)
At the start: 2 copper layers, 21.5 x 37 mm, 8 parts, among them J1 MD-40SM, M1 Module_XIAO-ESP32S3, Q1 BSS138

Commit message: corrected layout with two unconnected nets (oops)
Routing:
- net 3.3V: track 31.3 -> 48.3 mm, vias 0 -> 1
- net 5V: track 28.5 -> 37.3 mm
- net /ADB_1: track 22.6 -> 23.5 mm
Changed lines of the file:
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@@
 	)
 	(segment
-		(start 154.02 89.455)
-		(end 154.02 108.08)
+		(start 148.4 110.005)
+		(end 148.4 113.7)
+		(width 0.2)
+		(layer "F.Cu")
+		(net "5V")
+	)
+	(segment
+		(start 151.3 108.605)
+		(end 149.8 108.605)
+		(width 0.2)
+		(layer "F.Cu")
+		(net "5V")
+	)
+	(segment
+		(start 152 109.305)
+		(end 151.3 108.605)
+		(width 0.2)
+		(layer "F.Cu")
+		(net "5V")
+	)
+	(segment
+		(start 149.8 108.605)
+		(end 148.4 110.005)
+		(width 0.2)
+		(layer "F.Cu")
+		(net "5V")
+	)
+	(segment
+		(start 153.45 88.885)
+		(end 154.8 90.235)
 		(width 0.4)
 		(layer "B.Cu")
@@
 	)
 	(segment
-		(start 153.45 88.885)
-		(end 154.02 89.455)
-		(width 0.4)
-		(layer "B.Cu")
-		(net "5V")
-	)
-	(segment
-		(start 154.02 108.08)
+		(start 154.8 90.235)
+		(end 154.800001 107.299999)
+		(width 0.4)
+		(layer "B.Cu")
+		(net "5V")
+	)
+	(segment
+		(start 154.800001 107.299999)
 		(end 148.4 113.7)
 		(width 0.4)
@@
 	)
 	(segment
-		(start 150.5 109.305)
-		(end 149 110.805)
-		(width 0.2)
-		(layer "F.Cu")
-		(net "/ADB_1")
-	)
-	(segment
 		(start 149 110.805)
-		(end 146.5 110.805)
+		(end 150.5 109.305)
 		(width 0.2)
 		(layer "F.Cu")
@@
 	)
 	(segment
-		(start 142 109.905)
+		(start 141.4 110.405)
 		(end 141.4 109.305)
 		(width 0.2)
@@
 	)
 	(segment
-		(start 142 110.805)
-		(end 142 109.905)
+		(start 141 110.805)
+		(end 141.4 110.405)
 		(width 0.2)
 		(layer "F.Cu")
@@
 	)
 	(via
-		(at 142 110.805)
+		(at 141 110.805)
 		(size 0.6)
 		(drill 0.3)
@@
 	)
 	(via
-		(at 146.5 110.805)
+		(at 149 110.805)
 		(size 0.6)
 		(drill 0.3)
@@
 	)
 	(segment
-		(start 146.5 110.805)
-		(end 142 110.805)
-		(width 0.2)
-		(layer "B.Cu")
-		(net "/ADB_1")
+		(start 149 110.805)
+		(end 141 110.805)
+		(width 0.2)
+		(layer "B.Cu")
+		(net "/ADB_1")
+	)
+	(segment
+		(start 152.8 114.008)
+		(end 149.504 117.304)
+		(width 0.4)
+		(layer "F.Cu")
+		(net "3.3V")
+	)
+	(segment
+		(start 154 107)
+		(end 154 107.305)
+		(width 0.4)
+		(layer "F.Cu")
+		(net "3.3V")
+	)
+	(segment
+		(start 145.1 110.205)
+		(end 146 109.305)
+		(width 0.4)
+		(layer "F.Cu")
+		(net "3.3V")
+	)
+	(segment
+		(start 145.1 115.108)
+		(end 145.1 110.205)
+		(width 0.4)
+		(layer "F.Cu")
+		(net "3.3V")
+	)
+	(segment
+		(start 149.504 117.304)
+		(end 147.296 117.304)
+		(width 0.4)
+		(layer "F.Cu")
+		(net "3.3V")
+	)
+	(segment
+		(start 152.8 108.505)
+		(end 152.8 114.008)
+		(width 0.4)
+		(layer "F.Cu")
+		(net "3.3V")
+	)
+	(segment
+		(start 147.296 117.304)
+		(end 145.1 115.108)
+		(width 0.4)
+		(layer "F.Cu")
+		(net "3.3V")
 	)
 	(segment
@@
 	)
 	(segment
+		(start 154 107.305)
+		(end 152.8 108.505)
+		(width 0.4)
+		(layer "F.Cu")
+		(net "3.3V")
+	)
+	(segment
 		(start 146 109.305)
 		(end 145.1 108.405)
@@
 		(net "3.3V")
 	)
-	(segment
-		(start 152.32 93.965)
-		(end 153.42 95.065)
-		(width 0.4)
-		(layer "B.Cu")
-		(net "3.3V")
-	)
-	(segment
-		(start 148.695635 109.305)
-		(end 146 109.305)
-		(width 0.4)
-		(layer "B.Cu")
-		(net "3.3V")
-	)
-	(segment
-		(start 153.42 95.065)
-		(end 153.42 104.580635)
-		(width 0.4)
-		(layer "B.Cu")
-		(net "3.3V")
-	)
-	(segment
-		(start 153.42 104.580635)
-		(end 148.695635 109.305)
+	(via
+		(at 154 107)
+		(size 0.6)
+		(drill 0.3)
+		(layers "F.Cu" "B.Cu")
+		(net "3.3V")
+	)
+	(segment
+		(start 154 95.645)
+		(end 152.32 93.965)
+		(width 0.4)
+		(layer "B.Cu")
+		(net "3.3V")
+	)
+	(segment
+		(start 154 107)
+		(end 154 95.645)
 		(width 0.4)
 		(layer "B.Cu")
@@
 		(fill yes
 			(thermal_gap 0.5)
-			(thermal_bridge_width 0.5)
+			(thermal_bridge_width 0.25)
 			(smoothing fillet)
 			(radius 2)
@@
 		(fill yes
 			(thermal_gap 0.5)
-			(thermal_bridge_width 0.5)
+			(thermal_bridge_width 0.25)
 			(smoothing fillet)
 			(radius 2)
